Commit message: Revamped the robot model: static objects are excluded.

File: anobot_description/urdf/anobot.urdf.xacro (robot description, xacro)
@@ -1,5 +1,4 @@
 <?xml version="1.0"?>
-<robot name="anobot_cell" xmlns:xacro="http://ros.org/wiki/xacro">
-  <xacro:include filename="$(find anobot_description)/urdf/anobot_env.xacro"/>
+<robot name="anobot" xmlns:xacro="http://ros.org/wiki/xacro">
   <xacro:include filename="$(find anobot_description)/urdf/anobot_agv.xacro"/>
   <xacro:include filename="$(find anobot_description)/urdf/anobot_ur.xacro"/>
@@ -28,18 +27,4 @@
     <color rgba="0.60 0.98 0.60 1"/>
   </material>
-  <link name="world"/>
-  <xacro:workstation
-    name="workstation_1"
-    parent="world"
-    >
-    <origin xyz="0 1.5 0" rpy="0 0 0"/>
-  </xacro:workstation>
-  <!-- TEMPORARY RVIZ FIX: Connect the world to the AGV so it builds a single root tree -->
-  <!-- Remove or comment this joint out when moving to Gazebo/Nav2! -->
-  <joint name="rviz_temporary_world_to_agv" type="fixed">
-    <parent link="world"/>
-    <child link="base_footprint"/>
-    <origin xyz="0 0 0" rpy="0 0 0"/>
-  </joint>
   <xacro:anobot_agv/>
   <xacro:anobot_ur
@@ -49,13 +34,11 @@
     kinematics_parameters_file="$(arg kinematics_parameters_file)"
     physical_parameters_file="$(arg physical_parameters_file)"
-    visual_parameters_file="$(arg visual_parameters_file)"
-    >
-    <origin xyz="0 0 0" rpy="0 0 0" />
+    visual_parameters_file="$(arg visual_parameters_file)">
+    <origin xyz="0 0 0" rpy="0 0 0"/>
   </xacro:anobot_ur>
   <xacro:anobot_end_effector
     ur_type="$(arg ur_type)"
-    connected_to="tool0"
-    >
-    <origin xyz="0 0 0" rpy="0 0 0" />
+    connected_to="tool0">
+    <origin xyz="0 0 0" rpy="0 0 0"/>
   </xacro:anobot_end_effector>
 </robot>

File: anobot_description/urdf/anobot_agv.xacro (robot description, xacro)
@@ -1,19 +1,21 @@
 <?xml version="1.0"?>
 <robot xmlns:xacro="http://ros.org/wiki/xacro">
-  <!-- <xacro:macro name="anobot_agv" params="parent"> -->
   <xacro:macro name="anobot_agv">
-    <xacro:property name="ground_clearance" value="0.050" />
-    <xacro:property name="agv_length" value="0.936" />
-    <xacro:property name="agv_width" value="0.630" />
-    <xacro:property name="agv_height" value="0.215" />
-    <xacro:property name="body_length" value="0.9" />
-    <xacro:property name="body_width" value="0.6" />
-    <xacro:property name="body_height" value="0.6" />
-    <link name="base_footprint" />
+    <xacro:property name="ground_clearance" value="0.050"/>
+    <xacro:property name="agv_length" value="0.936"/>
+    <xacro:property name="agv_width" value="0.630"/>
+    <xacro:property name="agv_height" value="0.215"/>
+    <xacro:property name="body_length" value="0.9"/>
+    <xacro:property name="body_width" value="0.6"/>
+    <xacro:property name="body_height" value="0.6"/>
+    <link name="base_footprint"/>
     <link name="base_link">
       <inertial>
-        <origin xyz="0 0 0" rpy="0 0 0" />
-        <mass value="65.0" />
-        <inertia ixx="3.2" ixy="0.0" ixz="0.0" iyy="5.2" iyz="0.0" izz="6.7"/>
+        <origin xyz="0 0 0" rpy="0 0 0"/>
+        <mass value="65.0"/>
+        <inertia
+          ixx="3.2" ixy="0.0" ixz="0.0"
+          iyy="5.2" iyz="0.0"
+          izz="6.7"/>
       </inertial>
       <visual>
@@ -49,5 +51,5 @@
       <visual>
         <geometry>
-          <mesh filename="package://anobot_description/meshes/estop.dae" scale="1 1 1" />
+          <mesh filename="package://anobot_description/meshes/estop.dae" scale="1 1 1"/>
         </geometry>
         <origin rpy="0 0 0" xyz="0 0 0"/>
@@ -58,17 +60,17 @@
       <parent link="base_footprint"/>
       <child link="base_link"/>
-      <origin xyz="0 0 ${agv_height/2+ground_clearance}" rpy="0 0 0"/>
+      <origin xyz="0 0 ${agv_height/2 + ground_clearance}" rpy="0 0 0"/>
     </joint>
-    <joint name="base_to_body" type="fixed">
+    <joint name="base_link_to_body_link" type="fixed">
       <parent link="base_link"/>
       <child link="body_link"/>
-      <origin xyz="0 0 ${agv_height/2+body_height/2}" rpy="0 0 0"/>
+      <origin xyz="0 0 ${agv_height/2 + body_height/2}" rpy="0 0 0"/>
     </joint>
-    <joint name="body_to_estop" type="fixed">
+    <joint name="body_link_to_dummy_estop" type="fixed">
       <parent link="body_link"/>
       <child link="dummy_estop"/>
-      <origin xyz="0 ${-body_width/2+0.030} ${body_height/2-0.050}" rpy="0 0 3.1416"/>
+      <origin xyz="0 ${-body_width/2 + 0.030} ${body_height/2 - 0.050}" rpy="0 0 3.1416"/>
     </joint>
-    <joint name="body_to_mount" type="fixed">
+    <joint name="body_link_to_robot_mount" type="fixed">
       <parent link="body_link"/>
       <child link="robot_mount"/>

File: anobot_description/urdf/anobot_end_effector.xacro (robot description, xacro)
@@ -1,4 +1,4 @@
 <?xml version="1.0" encoding="utf-8"?>
-<robot xmlns:xacro="https://ros.org/wiki/xacro">
+<robot xmlns:xacro="http://ros.org/wiki/xacro">
   <xacro:macro name="anobot_end_effector" params="
   ur_type

File: anobot_description/urdf/anobot_ur.xacro (robot description, xacro)
@@ -10,15 +10,14 @@
     visual_parameters_file
     *origin
-    ">
+  ">
     <xacro:ur_robot
       name="${ur_type}"
       tf_prefix="${ur_type}_"
-      parent="robot_mount"
+      parent="${parent}"
       joint_limits_parameters_file="${joint_limits_parameters_file}"
       kinematics_parameters_file="${kinematics_parameters_file}"
       physical_parameters_file="${physical_parameters_file}"
-      visual_parameters_file="${visual_parameters_file}"
-    >
-      <origin xyz="0 0 0" rpy="0 0 0" />
+      visual_parameters_file="${visual_parameters_file}">
+      <xacro:insert_block name="origin"/>
     </xacro:ur_robot>
   </xacro:macro>

File: anobot_ur_bridge/urdf/anobot_ur_bridge.urdf.xacro (robot description, xacro)
@@ -1,5 +1,4 @@
 <?xml version="1.0"?>
-<robot name="anobot_cell" xmlns:xacro="http://ros.org/wiki/xacro">
-  <xacro:include filename="$(find anobot_description)/urdf/anobot_env.xacro"/>
+<robot name="anobot" xmlns:xacro="http://ros.org/wiki/xacro">
   <xacro:include filename="$(find anobot_description)/urdf/anobot_agv.xacro"/>
   <xacro:include filename="$(find anobot_description)/urdf/anobot_ur.xacro"/>
@@ -29,18 +28,4 @@
     <color rgba="0.60 0.98 0.60 1"/>
   </material>
-  <link name="world"/>
-  <xacro:workstation
-    name="workstation_1"
-    parent="world"
-    >
-    <origin xyz="0 1.5 0" rpy="0 0 0"/>
-  </xacro:workstation>
-  <!-- TEMPORARY RVIZ FIX: Connect the world to the AGV so it builds a single root tree -->
-  <!-- Remove or comment this joint out when moving to Gazebo/Nav2! -->
-  <joint name="rviz_temporary_world_to_agv" type="fixed">
-    <parent link="world"/>
-    <child link="base_footprint"/>
-    <origin xyz="0 0 0" rpy="0 0 0"/>
-  </joint>
   <xacro:anobot_agv/>
   <xacro:anobot_ur
@@ -50,13 +35,11 @@
     kinematics_parameters_file="$(arg kinematics_parameters_file)"
     physical_parameters_file="$(arg physical_parameters_file)"
-    visual_parameters_file="$(arg visual_parameters_file)"
-    >
-    <origin xyz="0 0 0" rpy="0 0 0" />
+    visual_parameters_file="$(arg visual_parameters_file)">
+    <origin xyz="0 0 0" rpy="0 0 0"/>
   </xacro:anobot_ur>
   <xacro:anobot_end_effector
     ur_type="$(arg ur_type)"
-    connected_to="tool0"
-    >
-    <origin xyz="0 0 0" rpy="0 0 0" />
+    connected_to="tool0">
+    <origin xyz="0 0 0" rpy="0 0 0"/>
   </xacro:anobot_end_effector>
   <xacro:arg name="robot_ip" default="192.168.56.101"/>
