Commit message: feat: integrate UR10e camera mount and validate MoveIt mock control - refactor robot description into reusable Xacro macros - add D435i camera and tool-mount frames - standardize UR link and joint prefixing - add ros2_control wrapper and MoveIt configuration - validate TF, mock trajectory execution, and ArUco repeatability

File: anobot_description/urdf/anobot.urdf.xacro (robot description, xacro)
@@ -1,44 +1,21 @@
 <?xml version="1.0"?>
 <robot name="anobot" xmlns:xacro="http://ros.org/wiki/xacro">
-  <xacro:include filename="$(find anobot_description)/urdf/anobot_agv.xacro"/>
-  <xacro:include filename="$(find anobot_description)/urdf/anobot_ur.xacro"/>
-  <xacro:include filename="$(find anobot_description)/urdf/anobot_end_effector.xacro"/>
+  <xacro:include filename="$(find anobot_description)/urdf/anobot_macro.xacro"/>
   <xacro:arg name="ur_type" default="ur10e"/>
-  <xacro:arg name="joint_limits_parameters_file" default="$(find ur_description)/config/$(arg ur_type)/joint_limits.yaml"/>
-  <xacro:arg name="kinematics_parameters_file" default="$(find ur_description)/config/$(arg ur_type)/default_kinematics.yaml"/>
-  <xacro:arg name="physical_parameters_file" default="$(find ur_description)/config/$(arg ur_type)/physical_parameters.yaml"/>
-  <xacro:arg name="visual_parameters_file" default="$(find ur_description)/config/$(arg ur_type)/visual_parameters.yaml"/>
-  <material name="dark_grey">
-     <color rgba="0.25 0.25 0.25 1"/>
-  </material>
-  <material name="grey">
-    <color rgba="0.5 0.5 0.5 1"/>
-  </material>
-  <material name="invisible">
-    <color rgba="0.9 0.9 0.9 0.1"/>
-  </material>
-  <material name="white">
-    <color rgba="1 1 1 1"/>
-  </material>
-  <material name="cobalt_blue">
-    <color rgba="0 0.25 0.76 1"/>
-  </material>
-  <material name="pale_green">
-    <color rgba="0.60 0.98 0.60 1"/>
-  </material>
-  <xacro:anobot_agv/>
-  <xacro:anobot_ur
-    parent="robot_mount"
+  <xacro:arg name="tf_prefix" default="ur_"/>
+  <xacro:arg name="joint_limits_parameters_file"
+    default="$(find ur_description)/config/$(arg ur_type)/joint_limits.yaml"/>
+  <xacro:arg name="kinematics_parameters_file"
+    default="$(find ur_description)/config/$(arg ur_type)/default_kinematics.yaml"/>
+  <xacro:arg name="physical_parameters_file"
+    default="$(find ur_description)/config/$(arg ur_type)/physical_parameters.yaml"/>
+  <xacro:arg name="visual_parameters_file"
+    default="$(find ur_description)/config/$(arg ur_type)/visual_parameters.yaml"/>
+  <xacro:anobot
     ur_type="$(arg ur_type)"
+    tf_prefix="$(arg tf_prefix)"
     joint_limits_parameters_file="$(arg joint_limits_parameters_file)"
     kinematics_parameters_file="$(arg kinematics_parameters_file)"
     physical_parameters_file="$(arg physical_parameters_file)"
-    visual_parameters_file="$(arg visual_parameters_file)">
-    <origin xyz="0 0 0" rpy="0 0 0"/>
-  </xacro:anobot_ur>
-  <xacro:anobot_end_effector
-    ur_type="$(arg ur_type)"
-    connected_to="tool0">
-    <origin xyz="0 0 0" rpy="0 0 0"/>
-  </xacro:anobot_end_effector>
+    visual_parameters_file="$(arg visual_parameters_file)"/>
 </robot>

File: anobot_description/urdf/anobot_agv.xacro (robot description, xacro)
@@ -48,5 +48,5 @@
       </collision>
     </link>
-    <link name="dummy_estop">
+    <link name="estop_link">
       <visual>
         <geometry>
@@ -67,13 +67,15 @@
       <origin xyz="0 0 ${agv_height/2 + body_height/2}" rpy="0 0 0"/>
     </joint>
-    <joint name="body_link_to_dummy_estop" type="fixed">
+    <joint name="estop_joint" type="fixed">
       <parent link="body_link"/>
-      <child link="dummy_estop"/>
-      <origin xyz="0 ${-body_width/2 + 0.030} ${body_height/2 - 0.050}" rpy="0 0 3.1416"/>
+      <child link="estop_link"/>
+      <!-- <origin xyz="0 ${-body_width/2.0 + 0.030} ${body_height/2.0 - 0.050}" rpy="0 0 ${pi}"/> -->
+      <origin xyz="0 ${body_width/2.0 - 0.030} ${body_height/2.0 - 0.050}" rpy="0 0 0"/>
     </joint>
     <joint name="body_link_to_robot_mount" type="fixed">
       <parent link="body_link"/>
       <child link="robot_mount"/>
-      <origin xyz="0 0 ${body_height/2}" rpy="0 0 -1.5708"/>
+      <!-- <origin xyz="0 0 ${body_height/2.0}" rpy="0 0 ${-pi/2.0}"/> -->
+      <origin xyz="0 0 ${body_height/2.0}" rpy="0 0 ${-pi}"/>
     </joint>
     <gazebo reference="base_link">

File: anobot_description/urdf/anobot_end_effector.xacro (robot description, xacro)
@@ -2,20 +2,18 @@
 <robot xmlns:xacro="http://ros.org/wiki/xacro">
   <xacro:macro name="anobot_end_effector" params="
-    ur_type
-    connected_to
+    parent
+    tool_link:=anobot_tool_link
+    grasp_frame:=anobot_grasp_frame
+    tool_length:=0.150
+    tool_width:=0.100
+    tool_depth:=0.100
+    tool_mass:=1.0
     *origin
   ">
     <!--
       Temporary end-effector envelope for workspace and collision studies.
-      tool_length:
-        Distance from UR tool0 to the assumed rod gripping point.
-      The dimensions should later be replaced with the actual end-effector
-      dimensions and calibrated grasp frame.
+      Replace with the actual end-effector geometry and mass properties.
     -->
-    <xacro:property name="tool_length" value="0.150"/>
-    <xacro:property name="tool_width" value="0.100"/>
-    <xacro:property name="tool_depth" value="0.100"/>
-    <!-- Physical placeholder end-effector -->
-    <link name="anobot_tool_link">
+    <link name="${tool_link}">
       <visual>
         <origin
@@ -35,10 +33,9 @@
         </geometry>
       </collision>
-      <!-- Inertial values are approximate and only for simulation validity. -->
       <inertial>
         <origin
           xyz="0 0 ${tool_length / 2.0}"
           rpy="0 0 0"/>
-        <mass value="1.0"/>
+        <mass value="${tool_mass}"/>
         <inertia
           ixx="0.002708"
@@ -50,17 +47,14 @@
       </inertial>
     </link>
-    <joint name="anobot_tool_joint" type="fixed">
-      <parent link="${ur_type}_${connected_to}"/>
-      <child link="anobot_tool_link"/>
-      <origin xyz="0 0 0" rpy="0 0 0"/>
+    <joint name="${tool_link}_joint" type="fixed">
+      <parent link="${parent}"/>
+      <child link="${tool_link}"/>
+      <xacro:insert_block name="origin"/>
     </joint>
-    <!--
-      This link is the assumed rod grasping point.
-      An attached MoveIt collision object can be attached to this link.
-    -->
-    <link name="anobot_grasp_frame"/>
-    <joint name="anobot_grasp_joint" type="fixed">
-      <parent link="anobot_tool_link"/>
-      <child link="anobot_grasp_frame"/>
+    <!-- Nominal task frame at the assumed rod gripping point. -->
+    <link name="${grasp_frame}"/>
+    <joint name="${grasp_frame}_joint" type="fixed">
+      <parent link="${tool_link}"/>
+      <child link="${grasp_frame}"/>
       <origin xyz="0 0 ${tool_length}" rpy="0 0 0"/>
     </joint>

File: anobot_description/urdf/anobot_ur.xacro (robot description, xacro)
@@ -5,4 +5,5 @@
     parent
     ur_type
+    tf_prefix
     joint_limits_parameters_file
     kinematics_parameters_file
@@ -13,5 +14,5 @@
     <xacro:ur_robot
       name="${ur_type}"
-      tf_prefix="${ur_type}_"
+      tf_prefix="${tf_prefix}"
       parent="${parent}"
       joint_limits_parameters_file="${joint_limits_parameters_file}"

File: anobot_ur_bridge/urdf/anobot_ur_bridge.urdf.xacro (robot description, xacro)
@@ -1,56 +1,36 @@
 <?xml version="1.0"?>
 <robot name="anobot" xmlns:xacro="http://ros.org/wiki/xacro">
-  <xacro:include filename="$(find anobot_description)/urdf/anobot_agv.xacro"/>
-  <xacro:include filename="$(find anobot_description)/urdf/anobot_ur.xacro"/>
-  <xacro:include filename="$(find anobot_description)/urdf/anobot_end_effector.xacro"/>
+  <xacro:include filename="$(find anobot_description)/urdf/anobot_macro.xacro"/>
   <xacro:include filename="$(find ur_robot_driver)/urdf/ur.ros2_control.xacro"/>
   <xacro:arg name="ur_type" default="ur10e"/>
-  <xacro:arg name="joint_limits_parameters_file" default="$(find ur_description)/config/$(arg ur_type)/joint_limits.yaml"/>
-  <xacro:arg name="kinematics_parameters_file" default="$(find ur_description)/config/$(arg ur_type)/default_kinematics.yaml"/>
-  <xacro:arg name="physical_parameters_file" default="$(find ur_description)/config/$(arg ur_type)/physical_parameters.yaml"/>
-  <xacro:arg name="visual_parameters_file" default="$(find ur_description)/config/$(arg ur_type)/visual_parameters.yaml"/>
-  <material name="dark_grey">
-     <color rgba="0.25 0.25 0.25 1"/>
-  </material>
-  <material name="grey">
-    <color rgba="0.5 0.5 0.5 1"/>
-  </material>
-  <material name="invisible">
-    <color rgba="0.9 0.9 0.9 0.1"/>
-  </material>
-  <material name="white">
-    <color rgba="1 1 1 1"/>
-  </material>
-  <material name="cobalt_blue">
-    <color rgba="0 0.25 0.76 1"/>
-  </material>
-  <material name="pale_green">
-    <color rgba="0.60 0.98 0.60 1"/>
-  </material>
-  <xacro:anobot_agv/>
-  <xacro:anobot_ur
-    parent="robot_mount"
+  <xacro:arg name="tf_prefix" default="ur_"/>
+  <xacro:arg name="joint_limits_parameters_file"
+    default="$(find ur_description)/config/$(arg ur_type)/joint_limits.yaml"/>
+  <xacro:arg name="kinematics_parameters_file"
+    default="$(find ur_description)/config/$(arg ur_type)/default_kinematics.yaml"/>
+  <xacro:arg name="physical_parameters_file"
+    default="$(find ur_description)/config/$(arg ur_type)/physical_parameters.yaml"/>
+  <xacro:arg name="visual_parameters_file"
+    default="$(find ur_description)/config/$(arg ur_type)/visual_parameters.yaml"/>
+  <xacro:arg name="robot_ip" default="192.168.56.101"/>
+  <xacro:arg name="headless_mode" default="false"/>
+  <xacro:arg name="use_mock_hardware" default="false"/>
+  <xacro:arg name="mock_sensor_commands" default="false"/>
+  <xacro:arg name="ur_script_filename"
+    default="$(find ur_client_library)/resources/external_control.urscript"/>
+  <xacro:arg name="ur_output_recipe_filename"
+    default="$(find ur_robot_driver)/resources/rtde_output_recipe.txt"/>
+  <xacro:arg name="ur_input_recipe_filename"
+    default="$(find ur_robot_driver)/resources/rtde_input_recipe.txt"/>
+  <xacro:anobot
     ur_type="$(arg ur_type)"
+    tf_prefix="$(arg tf_prefix)"
     joint_limits_parameters_file="$(arg joint_limits_parameters_file)"
     kinematics_parameters_file="$(arg kinematics_parameters_file)"
     physical_parameters_file="$(arg physical_parameters_file)"
-    visual_parameters_file="$(arg visual_parameters_file)">
-    <origin xyz="0 0 0" rpy="0 0 0"/>
-  </xacro:anobot_ur>
-  <xacro:anobot_end_effector
-    ur_type="$(arg ur_type)"
-    connected_to="tool0">
-    <origin xyz="0 0 0" rpy="0 0 0"/>
-  </xacro:anobot_end_effector>
-  <xacro:arg name="robot_ip" default="192.168.56.101"/>
-  <xacro:arg name="headless_mode" default="false" />
-  <xacro:arg name="ur_script_filename" default="$(find ur_client_library)/resources/external_control.urscript"/>
-  <xacro:arg name="ur_output_recipe_filename" default="$(find ur_robot_driver)/resources/rtde_output_recipe.txt"/>
-  <xacro:arg name="ur_input_recipe_filename" default="$(find ur_robot_driver)/resources/rtde_input_recipe.txt"/>
-  <xacro:arg name="use_mock_hardware" default="false" />
-  <xacro:arg name="mock_sensor_commands" default="false" />
+    visual_parameters_file="$(arg visual_parameters_file)"/>
   <xacro:ur_ros2_control
     name="$(arg ur_type)"
-    tf_prefix="$(arg ur_type)_"
+    tf_prefix="$(arg tf_prefix)"
     kinematics_parameters_file="$(arg kinematics_parameters_file)"
     robot_ip="$(arg robot_ip)"
@@ -60,5 +40,4 @@
     use_mock_hardware="$(arg use_mock_hardware)"
     mock_sensor_commands="$(arg mock_sensor_commands)"
-    headless_mode="$(arg headless_mode)"
-  />
+    headless_mode="$(arg headless_mode)"/>
 </robot>
