Commit message: Tested function to load entire anodizing line layout

File: anobot_description/urdf/anobot_agv.xacro (robot description, xacro)
@@ -3,10 +3,10 @@
   <xacro:macro name="anobot_agv">
     <xacro:property name="ground_clearance" value="0.050"/>
-    <xacro:property name="agv_length" value="0.936"/>
-    <xacro:property name="agv_width" value="0.630"/>
-    <xacro:property name="agv_height" value="0.215"/>
+    <xacro:property name="agv_length" value="1.034"/>
+    <xacro:property name="agv_width" value="0.680"/>
+    <xacro:property name="agv_height" value="0.320"/>
     <xacro:property name="body_length" value="0.9"/>
     <xacro:property name="body_width" value="0.6"/>
-    <xacro:property name="body_height" value="0.6"/>
+    <xacro:property name="body_height" value="0.9"/>
     <link name="base_footprint"/>
     <link name="base_link">

Commit message: feat: add calibrated workstation scene and grasp pose - apply UR10e factory kinematic calibration - integrate D435i eye-in-hand calibration - localize workstation marker in the robot base frame - add dummy tank visualization and collision geometry - add camera_view named state - define adjustable marker-relative grasp pose

File: anobot_description/urdf/anobot_agv.xacro (robot description, xacro)
@@ -2,11 +2,11 @@
 <robot xmlns:xacro="http://ros.org/wiki/xacro">
   <xacro:macro name="anobot_agv">
-    <xacro:property name="ground_clearance" value="0.050"/>
-    <xacro:property name="agv_length" value="1.034"/>
-    <xacro:property name="agv_width" value="0.680"/>
-    <xacro:property name="agv_height" value="0.320"/>
-    <xacro:property name="body_length" value="0.9"/>
-    <xacro:property name="body_width" value="0.6"/>
-    <xacro:property name="body_height" value="0.9"/>
+    <xacro:property name="ground_clearance" value="0.130"/>
+    <xacro:property name="agv_length" value="0.780"/>
+    <xacro:property name="agv_width" value="0.560"/>
+    <xacro:property name="agv_height" value="0.170"/>
+    <xacro:property name="body_length" value="0.780"/>
+    <xacro:property name="body_width" value="0.560"/>
+    <xacro:property name="body_height" value="0.880"/>
     <link name="base_footprint"/>
     <link name="base_link">

File: anobot_description/urdf/anobot_end_effector.xacro (robot description, xacro)
@@ -5,8 +5,6 @@
     tool_link:=anobot_tool_link
     grasp_frame:=anobot_grasp_frame
-    tool_length:=0.150
-    tool_width:=0.100
-    tool_depth:=0.100
-    tool_mass:=1.0
+    tool_length:=0.060
+    tool_mass:=0.150
     *origin
   ">
@@ -18,23 +16,25 @@
       <visual>
         <origin
-          xyz="0 0 ${tool_length / 2.0}"
-          rpy="0 0 0"/>
+          xyz="0 0 0"
+          rpy="${pi} 0 0"/>
         <geometry>
-          <box size="${tool_width} ${tool_depth} ${tool_length}"/>
+          <mesh
+            filename="package://anobot_description/meshes/60mm_stylus.STL"/>
         </geometry>
-        <material name="cobalt_blue"/>
+        <material name="white"/>
       </visual>
       <collision>
         <origin
-          xyz="0 0 ${tool_length / 2.0}"
-          rpy="0 0 0"/>
+          xyz="0 0 0"
+          rpy="${pi} 0 0"/>
         <geometry>
-          <box size="${tool_width} ${tool_depth} ${tool_length}"/>
+          <mesh
+            filename="package://anobot_description/meshes/60mm_stylus.STL"/>
         </geometry>
       </collision>
       <inertial>
         <origin
-          xyz="0 0 ${tool_length / 2.0}"
-          rpy="0 0 0"/>
+          xyz="0 0 0"
+          rpy="${pi} 0 0"/>
         <mass value="${tool_mass}"/>
         <inertia
